File: kicad/derek-cluster-controller-v3/derek_cluster_controller_revE_full_schematic.kicad_sch (KiCad schematic)
At the start: 75 parts, among them J1 5V DC INPUT, J13 I2C EXPANSION, J2 DEREK 1 RJ45 8P8C, J26 Teyleten Robot PCA9685 16ch S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, J3 DEREK 2 RJ45 8P8C, J4 DEREK 3 RJ45 8P8C, J5 DEREK 4 RJ45 8P8C, J6 DEREK 5 RJ45 8P8C, J7 DEREK 6 RJ45 8P8C, J8 DEREK 7 RJ45 8P8C, J9 DEREK 8 RJ45 8P8C, Q1 P-MOS REVERSE PROTECTION, SW1_1 DIP ID0, SW1_2 DIP ID1, SW1_3 DIP ID2, SW1_4 DIP ID3, U1 Hosyond ESP32-S3 N16R8 DevKit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, U3 WWZMDiB DFPlayer Mini #1, U4 WWZMDiB DFPlayer Mini #2, U5 74AHCT125 WS2812 level shifter

Commit message: KiCad PCB files for cluster controller
Parts:
- J26: value Teyleten Robot PCA9685 16ch Servo Module Socket -> Adafruit Product 815 PCA9685 16ch Servo Driver Socket; footprint ClusterCustom:Teyleten_PCA9685_16ch_Module_60x25mm_VERIFY -> ClusterActual:Adafruit_815_PCA9685_Breakout_CarrierSocket_VERIFY; symbol Cluster:TEYLETEN_PCA9685_MODULE_SOCKET -> Cluster:ADAFRUIT_815_PCA9685_MODULE_SOCKET
Other:
- note added: "Exact-part assumptions: Hosyond ESP32-S3 N16R8 dual USB-C DevKit, WWZMDiB DFPlayer Mini, Adafruit Product 815 PCA9685 62.5x25.4mm breakout, 0.96in SSD1306 OLED GND/VCC/SCL/SDA, shielded 90-degree RJ45 8P8C jacks."
- note removed: "Exact-part assumptions: Hosyond ESP32-S3 N16R8 dual USB-C DevKit, WWZMDiB DFPlayer Mini, Teyleten Robot PCA9685 60x25mm module, 0.96in SSD1306 OLED GND/VCC/SCL/SDA, shielded 90-degree RJ45 8P8C jacks."
Changed lines of the file:
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@@
   )
   (text "DEREK CLUSTER CONTROLLER REV E - FULL NET/PIN SCHEMATIC" (at 20.00 15.00 0) (effects (font (size 2.2 2.2) (thickness 0.14) bold)))
-  (text "Exact-part assumptions: Hosyond ESP32-S3 N16R8 dual USB-C DevKit, WWZMDiB DFPlayer Mini, Teyleten Robot PCA9685 60x25mm module, 0.96in SSD1306 OLED GND/VCC/SCL/SDA, shielded 90-degree RJ45 8P8C jacks." (at 20.00 22.00 0) (effects (font (size 1.0 1.0) (thickness 0.14))))
+  (text "Exact-part assumptions: Hosyond ESP32-S3 N16R8 dual USB-C DevKit, WWZMDiB DFPlayer Mini, Adafruit Product 815 PCA9685 62.5x25.4mm breakout, 0.96in SSD1306 OLED GND/VCC/SCL/SDA, shielded 90-degree RJ45 8P8C jacks." (at 20.00 22.00 0) (effects (font (size 1.0 1.0) (thickness 0.14))))
   (text "WARNING: Verify physical footprints by 1:1 print/test-fit before PCBWay fabrication. This schematic defines electrical nets and intended module pinouts." (at 20.00 27.00 0) (effects (font (size 1.0 1.0) (thickness 0.14) bold)))
   (symbol (lib_id "Cluster:CONN_2") (at 25.00 45.00 0) (unit 1) (exclude_from_sim no) (in_bom yes) (on_board yes) (dnp no)
@@
   (wire (pts (xy 130.92 152.62) (xy 125.92 152.62)) (stroke (width 0.18) (type default)))
   (global_label "GND" (shape input) (at 125.92 152.62 0) (effects (font (size 1.0 1.0) (thickness 0.12))))
-  (symbol (lib_id "Cluster:TEYLETEN_PCA9685_MODULE_SOCKET") (at 245.00 125.00 0) (unit 1) (exclude_from_sim no) (in_bom yes) (on_board yes) (dnp no)
+  (symbol (lib_id "Cluster:ADAFRUIT_815_PCA9685_MODULE_SOCKET") (at 245.00 125.00 0) (unit 1) (exclude_from_sim no) (in_bom yes) (on_board yes) (dnp no)
     (property "Reference" "J26" (at 245.00 117.00 0) (effects (font (size 1.27 1.27))))
-    (property "Value" "Teyleten Robot PCA9685 16ch Servo Module Socket" (at 245.00 133.00 0) (effects (font (size 1.27 1.27))))
-    (property "Footprint" "ClusterCustom:Teyleten_PCA9685_16ch_Module_60x25mm_VERIFY" (at 245.00 125.00 0) (effects (font (size 1.27 1.27)) hide))
+    (property "Value" "Adafruit Product 815 PCA9685 16ch Servo Driver Socket" (at 245.00 133.00 0) (effects (font (size 1.27 1.27))))
+    (property "Footprint" "ClusterActual:Adafruit_815_PCA9685_Breakout_CarrierSocket_VERIFY" (at 245.00 125.00 0) (effects (font (size 1.27 1.27)) hide))
     (pin "VCC")
     (pin "V+")
