File: kicad/derek-cluster-controller-v3/derek_cluster_controller_revG_tht_first.kicad_sch (KiCad schematic)
At the start: 75 parts, among them J1 5V DC INPUT, J13 I2C EXPANSION, J2 DEREK 1 RJ45 8P8C, J26 Adafruit Product 815 PCA9685 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, J3 DEREK 2 RJ45 8P8C, J4 DEREK 3 RJ45 8P8C, J5 DEREK 4 RJ45 8P8C, J6 DEREK 5 RJ45 8P8C, J7 DEREK 6 RJ45 8P8C, J8 DEREK 7 RJ45 8P8C, J9 DEREK 8 RJ45 8P8C, Q1 P-MOS REVERSE PROTECTION, SW1_1 DIP ID0, SW1_2 DIP ID1, SW1_3 DIP ID2, SW1_4 DIP ID3, U1 Hosyond ESP32-S3 N16R8 DevKit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, U3 WWZMDiB DFPlayer Mini #1, U4 WWZMDiB DFPlayer Mini #2, U5 74AHCT125 WS2812 level shifter

Commit message: Simplified design to limit SMD and DIP switches
Parts:
- U5: value 74AHCT125 WS2812 level shifter -> SN74AHCT125N DIP-14 WS2812 level shifter
Other:
- title: Derek Cluster Controller Rev E - Full Schematic -> Derek Cluster Controller Rev G - Through-Hole First
Changed lines of the file:
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@@
   (paper "A0")
   (title_block
-    (title "Derek Cluster Controller Rev E - Full Schematic")
+    (title "Derek Cluster Controller Rev G - Through-Hole First")
     (date "2026-07-01")
     (rev "Rev E full schematic")
@@
   (symbol (lib_id "Cluster:74AHCT125") (at 325.00 285.00 0) (unit 1) (exclude_from_sim no) (in_bom yes) (on_board yes) (dnp no)
     (property "Reference" "U5" (at 325.00 277.00 0) (effects (font (size 1.27 1.27))))
-    (property "Value" "74AHCT125 WS2812 level shifter" (at 325.00 293.00 0) (effects (font (size 1.27 1.27))))
+    (property "Value" "SN74AHCT125N DIP-14 WS2812 level shifter" (at 325.00 293.00 0) (effects (font (size 1.27 1.27))))
     (property "Footprint" "Package_SO:SOIC-14_3.9x8.7mm_P1.27mm" (at 325.00 285.00 0) (effects (font (size 1.27 1.27)) hide))
     (pin "1OE")
