File: kicad/cluster_split_kicad_revC/Cluster_Servo_Board/Cluster_Servo_Board.kicad_sch (KiCad schematic)
At the start: 13 parts, among them J1 LOGIC INTERCONNECT, J10 5V/GND INPUT A, J11 5V/GND INPUT B, J2 RJ45 DEREK 1, J3 RJ45 DEREK 2, J4 RJ45 DEREK 3, J5 RJ45 DEREK 4, J6 RJ45 DEREK 5, J7 RJ45 DEREK 6, J8 RJ45 DEREK 7, J9 RJ45 DEREK 8, U1 Adafruit PCA9685 PWM CH0..CH15, U2 74AHCT125

Commit message: Servo Controller board half routed with .4 traces to reduce loss
Parts:
- J2, J3, J4, J5, J6, J7, J8, J9: footprint (none) -> Connector_RJ:RJ45_Amphenol_54602-x08_Horizontal
Other:
- note added: "CLUSTER SERVO BOARD - REV C"
- note removed: "CLUSTER SERVO BOARD - REV B"

Commit message: Fixed RJ45 footprints on all, cleaned up routing, ready for a run at PCBWay
Parts:
- removed U2: 74AHCT125, symbol 74xx:74AHCT125
Other:
- note removed: "U2 - 74AHCT125N LED LEVEL SHIFTER"
Changed lines of the file:
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@@
-		)
-	)
-	(text "U2 - 74AHCT125N LED LEVEL SHIFTER"
-		(exclude_from_sim no)
-		(at 210.82 30.48 0)
-		(effects
-			(font
-				(size 2.032 2.032)
-				(thickness 0.4064)
-				(bold yes)
-			)
-			(justify left bottom)
 		)
 	)
@@
 		)
 	)
-	(label "LED_DATA_3V3"
-		(at 214.63 50.8 180)
-		(effects
-			(font
-				(size 1.27 1.27)
-			)
-			(justify right bottom)
-		)
-	)
 	(label "+3V3_LOGIC"
 		(at 63.5 45.72 0)
@@
 	(label "I2C_SCL"
 		(at 63.5 50.8 0)
-		(effects
-			(font
-				(size 1.27 1.27)
-			)
-			(justify left bottom)
-		)
-	)
-	(label "LED_5V"
-		(at 242.57 50.8 0)
 		(effects
 			(font
@@
 					(unit 1)
 				)
-			)
-		)
-	)
-	(symbol
-		(lib_id "74xx:74AHCT125")
-		(at 228.6 50.8 0)
-		(unit 1)
-		(body_style 1)
-		(exclude_from_sim no)
-		(in_bom yes)
-		(on_board yes)
-		(in_pos_files yes)
-		(dnp no)
-		(property "Reference" "U2"
-			(at 228.6 42.7482 0)
-			(show_name no)
-			(do_not_autoplace no)
-			(effects
-				(font
-					(size 1.27 1.27)
-				)
-			)
-		)
-		(property "Value" "74AHCT125"
-			(at 228.6 45.0596 0)
-			(show_name no)
-			(do_not_autoplace no)
-			(effects
-				(font
-					(size 1.27 1.27)
-				)
-			)
-		)
-		(property "Footprint" ""
-			(at 228.6 50.8 0)
-			(show_name no)
-			(do_not_autoplace no)
-			(effects
-				(font
-					(size 1.27 1.27)
-				)
-			)
-		)
-		(property "Datasheet" ""
-			(at 228.6 50.8 0)
-			(show_name no)
-			(do_not_autoplace no)
-			(effects
-				(font
-					(size 1.27 1.27)
-				)
-			)
-		)
-		(property "Description" ""
-			(at 228.6 50.8 0)
-			(show_name no)
-			(do_not_autoplace no)
-			(effects
-				(font
-					(size 1.27 1.27)
-				)
-			)
-		)
-		(pin "9"
-		)
-		(pin "2"
-		)
-		(pin "4"
-		)
-		(pin "7"
-		)
-		(pin "3"
-		)
-		(pin "1"
-		)
-		(pin "6"
-		)
-		(pin "5"
-		)
-		(pin "8"
-		)
-		(pin "11"
-		)
-		(pin "12"
-		)
-		(pin "10"
-		)
-		(pin "13"
-		)
-		(pin "14"
-		)
-		(instances
-			(project "Cluster_Servo_Board"
-				(path "/388a9e91-0f0e-433a-bd5f-a378c5ea05cf"
-					(reference "U2")
-					(unit 1)
-				)
