File: kicad/cluster_split_kicad_revC/Cluster_Logic_Board/Cluster_Logic_Board.kicad_pcb (KiCad board)
At the start: 2 copper layers, 160 x 100 mm, 29 parts, among them J1 POWER_5V, J10 JST_XH_8, J2 OLED_1x4, J3 PIR_LEFT, J4 PIR_CENTER, J5 PIR_RIGHT, SW1 DIPSW_4, U1 Hosyond ESP32-S3 N16R8 44-pin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, U2 WWZMDiB DFPlayer Mini, U3 WWZMDiB DFPlayer Mini

Commit message: Fixed RJ45 footprints on all, cleaned up routing, ready for a run at PCBWay - more
Parts:
- added M3: MountingHole_3.2mm_M3, MountingHole:MountingHole_3.2mm_M3, F.Cu at (81.5, 51.0)
- added M3: MountingHole_3.2mm_M3, MountingHole:MountingHole_3.2mm_M3, F.Cu at (154.5, 5.50)
- added M3: MountingHole_3.2mm_M3, MountingHole:MountingHole_3.2mm_M3, F.Cu at (6.00, 94.0)
- added M3: MountingHole_3.2mm_M3, MountingHole:MountingHole_3.2mm_M3, F.Cu at (5.50, 5.00)
- added M3: MountingHole_3.2mm_M3, MountingHole:MountingHole_3.2mm_M3, F.Cu at (154.5, 94.5)

Commit message: Fixed servo controller footprint, submitted to JLCPCB today
Parts:
- added REF**: Jack_3.5mm_CUI_SJ1-3525N_Horizontal, Connector_Audio:Jack_3.5mm_CUI_SJ1-3525N_Horizontal, F.Cu at (181.0, 84.0)
- U2 - R DFPlayer: renamed from U2
- U3 - LEFT DFPlayer: renamed from U3
- moved U1 33.4 mm to (131.8, 61.9)
- moved U3 - LEFT DFPlayer 33.4 mm to (172.3, 66.1)
- moved C1 33.4 mm to (42.5, 50.5)
- moved C2 33.4 mm to (155.7, 71.5)
- moved C3 33.4 mm to (156.2, 75.0)
- moved C4 33.4 mm to (155.5, 104.0)
- moved C5 33.4 mm to (155.5, 109.0)
- moved C7 33.4 mm to (139.5, 108.0)
- moved C8 33.4 mm to (107.5, 88.0)
- moved J1 33.4 mm to (42.5, 39.5)
- moved J10 33.4 mm to (43.5, 81.8)
- moved J2 33.4 mm to (99.8, 56.5)
- moved J3 33.4 mm to (121.5, 111.5)
- moved J4 33.4 mm to (102.5, 112.0)
- moved J5 33.4 mm to (83.5, 111.5)
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Routing:
- net (no net): track 0.00 -> 47.0 mm
- net +3V3_LOGIC: track 158.9 -> 155.7 mm, vias 1 -> 0
Other:
- board text added: "CLUSTER LOGIC BOARD - REV H"
- board text removed: "CLUSTER LOGIC BOARD - REV G U1 REBUILT"
